File: PCB/OS3M_Mouse.kicad_sch (KiCad schematic)
At the start: 47 parts, among them J1 DBG_HDR, J2 USB_C_Receptacle_USB2.0, J3 EXP_HDR, SW1 SW_Push, U1 AP2112K-3.3, U2 LDC1614, U3 STM32F042F6P6, U4 LDC1612, U5 USBLC6-2SC6, X1 ASV-40.000MHz

Commit message: Swapped inner layers to get GND plane close to components, fixed shorted UART
Parts:
- added TP1, TP2, TP3, TP4: TestPoint, TestPoint:TestPoint_Pad_D1.0mm, symbol Connector:TestPoint
Connections:
- net at U3.10 (PA4): now also TP1.1
- net at U3.11 (PA5): now also TP2.1
- net at U3.12 (PA6): now also TP3.1
- net at U3.13 (PA7): now also TP4.1
- no-connect marks 9 -> 5
