File: PCB/OS3M_Mouse.kicad_sch (KiCad schematic)
At the start: 47 parts, among them J1 DBG_HDR, J2 USB_C_Receptacle_USB2.0, J3 EXP_HDR, SW1 SW_Push, U1 AP2112K-3.3, U2 LDC1614, U3 STM32F042F6P6, U4 LDC1612, U5 USBLC6-2SC6, X1 ASV-40.000MHz

Commit message: Update to Rev2, JLC manufacturable
Parts:
- added TP1, TP2, TP3, TP4: TestPoint, TestPoint:TestPoint_Pad_D2.0mm, symbol Connector:TestPoint
- J2: footprint Connector_USB:USB_C_Receptacle_GCT_USB4085 -> Connector_USB:USB_C_Receptacle_XKB_U262-16XN-4BVC11
Connections:
- net GND: now also U3.1 (PB8)
- net at U3.10 (PA4): now also TP1.1
- net at U3.11 (PA5): now also TP2.1
- net at U3.12 (PA6): now also TP3.1
- net at U3.13 (PA7): now also TP4.1
- no-connect marks 9 -> 4
Changed lines of the file:
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@@
   (junction (at 90.17 27.94) (diameter 0) (color 0 0 0 0)
   )
-  (no_connect (at 111.76 92.71))
-  (no_connect (at 111.76 95.25))
-  (no_connect (at 111.76 97.79))
-  (no_connect (at 111.76 100.33))
   (no_connect (at 81.28 107.95))
-  (no_connect (at 81.28 110.49))
   (no_connect (at 71.12 168.91))
   (no_connect (at 71.12 166.37))
@@
     (stroke (width 0) (type default) (color 0 0 0 0))
   )
+  (wire (pts (xy 111.76 92.71) (xy 123.19 92.71))
+    (stroke (width 0) (type default) (color 0 0 0 0))
+  )
   (polyline (pts (xy 143.51 53.34) (xy 143.51 125.73))
     (stroke (width 0) (type default) (color 0 0 0 0))
@@
     (stroke (width 0) (type default) (color 0 0 0 0))
   )
+  (wire (pts (xy 111.76 97.79) (xy 123.19 97.79))
+    (stroke (width 0) (type default) (color 0 0 0 0))
+  )
   (wire (pts (xy 210.82 138.43) (xy 223.52 138.43))
     (stroke (width 0) (type default) (color 0 0 0 0))
@@
     (stroke (width 0) (type default) (color 0 0 0 0))
   )
+  (wire (pts (xy 81.28 110.49) (xy 80.01 110.49))
+    (stroke (width 0) (type default) (color 0 0 0 0))
+  )
   (wire (pts (xy 91.44 63.5) (xy 91.44 76.2))
     (stroke (width 0) (type default) (color 0 0 0 0))
@@
     (stroke (width 0) (type default) (color 0 0 0 0))
   )
+  (wire (pts (xy 80.01 110.49) (xy 80.01 113.03))
+    (stroke (width 0) (type default) (color 0 0 0 0))
+  )
+  (wire (pts (xy 111.76 100.33) (xy 123.19 100.33))
+    (stroke (width 0) (type default) (color 0 0 0 0))
+  )
   (wire (pts (xy 91.44 76.2) (xy 93.98 76.2))
     (stroke (width 0) (type default) (color 0 0 0 0))
@@
   )
   (wire (pts (xy 248.92 133.35) (xy 264.16 133.35))
+    (stroke (width 0) (type default) (color 0 0 0 0))
+  )
+  (wire (pts (xy 111.76 95.25) (xy 123.19 95.25))
     (stroke (width 0) (type default) (color 0 0 0 0))
   )
@@
     )
     (property "Datasheet" "" (id 3) (at 236.22 26.67 0)
+      (effects (font (size 1.27 1.27)) hide)
+    )
+    (pin "1")
+  )
+  (symbol (lib_id "Connector:TestPoint") (at 123.19 92.71 270) (unit 1)
+    (in_bom yes) (on_board yes)
+    (property "Reference" "TP1" (id 0) (at 128.27 92.71 90)
+      (effects (font (size 1.27 1.27)) (justify left))
+    )
+    (property "Value" "TestPoint" (id 1) (at 132.08 92.71 90)
+      (effects (font (size 1.27 1.27)) (justify left) hide)
+    )
+    (property "Footprint" "TestPoint:TestPoint_Pad_D2.0mm" (id 2) (at 123.19 97.79 0)
+      (effects (font (size 1.27 1.27)) hide)
+    )
+    (property "Datasheet" "~" (id 3) (at 123.19 97.79 0)
       (effects (font (size 1.27 1.27)) hide)
     )
@@
     (property "Reference" "J2" (id 0) (at 64.77 134.62 0))
     (property "Value" "USB_C_Receptacle_USB2.0" (id 1) (at 44.45 158.75 90))
-    (property "Footprint" "Connector_USB:USB_C_Receptacle_GCT_USB4085" (id 2) (at 59.69 153.67 0)
+    (property "Footprint" "Connector_USB:USB_C_Receptacle_XKB_U262-16XN-4BVC11" (id 2) (at 59.69 153.67 0)
       (effects (font (size 1.27 1.27)) hide)
     )
@@
     (pin "S1")
   )
+  (symbol (lib_id "Connector:TestPoint") (at 123.19 97.79 270) (unit 1)
+    (in_bom yes) (on_board yes)
+    (property "Reference" "TP3" (id 0) (at 128.27 97.79 90)
+      (effects (font (size 1.27 1.27)) (justify left))
+    )
+    (property "Value" "TestPoint" (id 1) (at 132.08 97.79 90)
+      (effects (font (size 1.27 1.27)) (justify left) hide)
+    )
+    (property "Footprint" "TestPoint:TestPoint_Pad_D2.0mm" (id 2) (at 123.19 102.87 0)
+      (effects (font (size 1.27 1.27)) hide)
+    )
+    (property "Datasheet" "~" (id 3) (at 123.19 102.87 0)
+      (effects (font (size 1.27 1.27)) hide)
+    )
+    (pin "1")
+  )
   (symbol (lib_id "power:GND") (at 95.25 156.21 0) (unit 1)
     (in_bom yes) (on_board yes)
@@
     (pin "1")
   )
+  (symbol (lib_id "Connector:TestPoint") (at 123.19 100.33 270) (unit 1)
+    (in_bom yes) (on_board yes)
+    (property "Reference" "TP4" (id 0) (at 128.27 100.33 90)
+      (effects (font (size 1.27 1.27)) (justify left))
+    )
+    (property "Value" "TestPoint" (id 1) (at 132.08 100.33 90)
+      (effects (font (size 1.27 1.27)) (justify left) hide)
+    )
+    (property "Footprint" "TestPoint:TestPoint_Pad_D2.0mm" (id 2) (at 123.19 105.41 0)
+      (effects (font (size 1.27 1.27)) hide)
+    )
+    (property "Datasheet" "~" (id 3) (at 123.19 105.41 0)
+      (effects (font (size 1.27 1.27)) hide)
+    )
+    (pin "1")
+  )
   (symbol (lib_id "Device:C") (at 81.28 33.02 0) (unit 1)
     (in_bom yes) (on_board yes)
@@
     (pin "1")
     (pin "2")
+  )
+  (symbol (lib_id "power:GND") (at 80.01 113.03 0) (unit 1)
+    (in_bom yes) (on_board yes)
+    (property "Reference" "#PWR029" (id 0) (at 80.01 119.38 0)
+      (effects (font (size 1.27 1.27)) hide)
+    )
+    (property "Value" "GND" (id 1) (at 80.01 116.84 0))
+    (property "Footprint" "" (id 2) (at 80.01 113.03 0)
+      (effects (font (size 1.27 1.27)) hide)
+    )
+    (property "Datasheet" "" (id 3) (at 80.01 113.03 0)
+      (effects (font (size 1.27 1.27)) hide)
+    )
+    (pin "1")
   )
   (symbol (lib_id "power:GND") (at 69.85 40.64 0) (unit 1)
@@
     (pin "2")
   )
+  (symbol (lib_id "Connector:TestPoint") (at 123.19 95.25 270) (unit 1)
+    (in_bom yes) (on_board yes)
+    (property "Reference" "TP2" (id 0) (at 128.27 95.25 90)
+      (effects (font (size 1.27 1.27)) (justify left))
+    )
+    (property "Value" "TestPoint" (id 1) (at 132.08 95.25 90)
+      (effects (font (size 1.27 1.27)) (justify left) hide)
+    )
+    (property "Footprint" "TestPoint:TestPoint_Pad_D2.0mm" (id 2) (at 123.19 100.33 0)
+      (effects (font (size 1.27 1.27)) hide)
+    )
+    (property "Datasheet" "~" (id 3) (at 123.19 100.33 0)
+      (effects (font (size 1.27 1.27)) hide)
+    )
+    (pin "1")
+  )
   (symbol (lib_id "Device:LED") (at 110.49 33.02 90) (unit 1)
     (in_bom yes) (on_board yes)
@@
       (reference "#PWR028") (unit 1) (value "GND") (footprint "")
     )
+    (path "/a773078e-5aa4-43b7-98bd-d8df1cab7e12"
+      (reference "#PWR029") (unit 1) (value "GND") (footprint "")
+    )
     (path "/9d198824-18fd-4ffc-a3d0-d9fded136de8"
       (reference "#PWR0101") (unit 1) (value "VBUS") (footprint "")
@@
     )
     (path "/603bb607-41f9-418c-839c-76284ba8d2ab"
-      (reference "J2") (unit 1) (value "USB_C_Receptacle_USB2.0") (footprint "Connector_USB:USB_C_Receptacle_GCT_USB4085")
+      (reference "J2") (unit 1) (value "USB_C_Receptacle_USB2.0") (footprint "Connector_USB:USB_C_Receptacle_XKB_U262-16XN-4BVC11")
     )
     (path "/86be4490-3d74-4a19-b871-5d0876e1aae5"
@@
       (reference "SW1") (unit 1) (value "SW_Push") (footprint "Button_Switch_SMD:SW_SPST_TL3305A")
     )
+    (path "/2a8ad124-7b4d-4854-9bf6-9f76d089af50"
+      (reference "TP1") (unit 1) (value "TestPoint") (footprint "TestPoint:TestPoint_Pad_D2.0mm")
+    )
+    (path "/de3512ee-fcb6-42bb-a305-e79a97bd637f"
+      (reference "TP2") (unit 1) (value "TestPoint") (footprint "TestPoint:TestPoint_Pad_D2.0mm")
+    )
+    (path "/61087d09-5423-4855-ad89-6ed0609dbda4"
+      (reference "TP3") (unit 1) (value "TestPoint") (footprint "TestPoint:TestPoint_Pad_D2.0mm")
+    )
+    (path "/a4e2a544-84b3-4f52-82de-57d5fa081149"
+      (reference "TP4") (unit 1) (value "TestPoint") (footprint "TestPoint:TestPoint_Pad_D2.0mm")
+    )
     (path "/b5636929-8ecb-402b-96ee-ceef16383502"
